File: hw/switchboard.kicad_sch (KiCad schematic)
At the start: 0 parts

Commit message: bla
Parts:
- added C1: 100nF, PCM_JLCPCB:C_0603, symbol PCM_JLCPCB-Capacitors:0603,100nF
- added D20: SS24, Diode_SMD:D_SMA, symbol Diode:SS24
- added J1: Conn_01x04_Pin, Connector_PinHeader_2.54mm:PinHeader_1x04_P2.54mm_Vertical, symbol Connector:Conn_01x04_Pin
- added J2: 2604-1104, custom:CONN4_2604-1104_WAG, symbol custom:2604-1104
- added J3: Conn_01x03_Pin, Connector_PinHeader_2.54mm:PinHeader_1x03_P2.54mm_Horizontal, symbol Connector:Conn_01x03_Pin
- added P1: ~, custom:IDC-TH_10P-P2.54-H-R2-C5-S2.54, symbol custom:IDC Box 2X5 2.54MM
- added R1, R2, R3, R4, R5, R6: 10kΩ, PCM_JLCPCB:R_0603, symbol PCM_JLCPCB-Resistors:0603,10kΩ
- added R7: 120Ω, PCM_JLCPCB:R_0603, symbol PCM_JLCPCB-Resistors:0603,120Ω
- added SW10: ~, custom:SW-TH_12P-P2.54_SMQP-06B-TP, symbol custom:SMQP-06B-TP
- added U1: YAAJ_BluePill_Part_Like, custom:YAAJ_BluePill_1, symbol custom:YAAJ_BluePill_Part_Like
- added U2: SP485EEN, PCM_JLCPCB:SOIC-8_L5.0-W4.0-P1.27-LS6.0-BL, symbol PCM_JLCPCB-Interface:Transceiver, RS485/422, 10Mbps, SP485EEN-L/TR
- added U3: ~, custom:CHINA_MP1584EN, symbol custom:CHINA_MP1584EN
Connections:
- new net: D20.2 (A), U3.2 (5V_POS)
- new net: J3.3 (Pin_3), R7.2
- new net +24V: J2.7 (4_1), J2.8 (4_2), P1.10, U3.4 (IN_POS)
- new net +3V3: R1.1, R2.1, R3.1, R4.1, U1.20 (3V3), U1.38 (3V3)
- new net +5V: C1.1, D20.1 (K), J1.2 (Pin_2), R6.1, U1.18 (5V), U2.8 (VCC)
- new net AUX_PROG_RX: J1.4 (Pin_4), U1.7 (PA10)
- new net AUX_PROG_TX: J1.3 (Pin_3), U1.6 (PA9)
- new net DIP0: SW10.1, U1.29 (PA4)
- new net DIP1: SW10.2, U1.30 (PA5)
- new net DIP2: SW10.3, U1.31 (PA6)
- new net DIP3: SW10.4, U1.32 (PA7)
- new net DIP4: SW10.5, U1.23 (PC14)
- new net FET_0: U1.33 (PB0)
- new net FET_1: U1.34 (PB1)
- new net FET_2: U1.11 (PB3)
- new net FET_3: U1.12 (PB4)
- new net FET_4: U1.13 (PB5)
- new net FET_5: U1.14 (PB6)
- new net FET_6: U1.15 (PB7)
- new net FET_7: U1.16 (PB8)
- new net GND: C1.2, J1.1 (Pin_1), J2.5 (3_1), J2.6 (3_2), P1.4, R5.1, SW10.10, SW10.11, SW10.12, SW10.8, SW10.9, U1.19 (GND), U1.39 (GND), U1.40 (GND), U2.5 (GND), U3.1 (5V_NEG), U3.3 (IN_NEG)
- new net RELAY_0: P1.1
- new net RELAY_1: P1.2
- new net RELAY_2: P1.3
- new net RELAY_3: P1.5
- new net RELAY_4: P1.6
- new net RELAY_5: P1.7
- new net RELAY_6: P1.8
- new net RELAY_7: P1.9
- new net RS485_DE: R2.2, U1.26 (PA1), U2.3 (DE)
- new net RS485_RE: R3.2, U1.25 (PA0), U2.2 (RE#)
- new net RS485_RX: R4.2, U1.28 (PA3), U2.1 (RO)
- new net RS485_TX: R1.2, U1.27 (PA2), U2.4 (DI)
- new net RS_485_A: J2.3 (2_1), J2.4 (2_2), R6.2, R7.1, U2.6 (A)
- new net RS_485_B: J2.1 (1_1), J2.2 (1_2), J3.2 (Pin_2), R5.2, U2.7 (B)
- no-connect marks 0 -> 18
Other:
- added sheet switches (switchees.kicad_sch)
